File: schematics/lora-esp32-s3-node/lora-esp32-s3-node.kicad_sch (KiCad schematic)
At the start: 5 parts, among them SW1 SW_Push, U1 ESP32-S3-WROOM-2

Commit message: WIP Schematics
Parts:
- added C3: 1 uF, symbol Device:C
- added R2: 10K, symbol Device:R
- added SW2: SW_Push, Package_DIP:DIP-8_W7.62mm, symbol Switch:SW_Push
Connections:
- net +3V3: now also R2.1
- net GND: now also C3.2, SW2.1
- net at R1.2, SW1.2, U1.3 (EN): now also C3.1
- net at U1.27 (IO0): now also R2.2, SW2.2
